Commit message: [modify] 80cm x 80cm の大きさに変更

File: pr2_practice_gazebo/models/urdf/ar_marker.urdf (robot description, URDF)
Before this commit: robot ar_marker, 1 links, 0 joints
Links:
- link marker_box: geometry collision mesh filename=package://pr2_practice_gazebo/models/meshes/ar_marker.dae scale=0.080 0.080 0.080; visual mesh filename=package://pr2_practice_gazebo/models/meshes/ar_marker.dae scale=0.080 0.080 0.080
